File: pcb_design/battery monitor circuit design/battery monitor circuit design.kicad_sch (KiCad schematic)
At the start: 1 part

Commit message: alright
Parts:
- added DS1: WC1602A, Display:WC1602A, symbol Display_Character:WC1602A
- added U1: LM7805CT, PCM_Package_TO_SOT_THT_AKL:TO-220-3_Vertical, symbol PCM_Voltage_Regulator_AKL:LM7805CT
- added U2: PCF8574, symbol Interface_Expansion:PCF8574
Connections:
- new net: DS1.10 (D3), U2.7 (P3)
- new net: DS1.11 (D4), U2.9 (P4)
- new net: DS1.12 (D5), U2.10 (P5)
- new net: DS1.13 (D6), U2.11 (P6)
- new net: DS1.14 (D7), U2.12 (P7)
- new net: DS1.7 (D0), U2.4 (P0)
- new net: DS1.8 (D1), U2.5 (P1)
- new net: DS1.9 (D2), U2.6 (P2)
